File: Hardware/Electrical/PCB_v2/Battery.kicad_sch (KiCad schematic)
At the start: 16 parts, among them J1 10k NTC, U1 BQ25303JRTER

Commit message: Components placed
Parts:
- C1, C5: value 2.2u -> 2.2uF
- C2, C3: value 10u -> 10uF
- C4: value 47n -> 47nF
- R6: value 0 -> 0 Ohm
- U1: *LCSC Part Number (none) -> C2842775
Changed lines of the file:
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@@
 			)
 		)
-		(property "Value" "10u"
+		(property "Value" "10uF"
 			(at 217.424 114.046 0)
 			(show_name no)
@@
 			)
 		)
-		(property "Value" "0"
+		(property "Value" "0 Ohm"
 			(at 160.02 145.542 90)
 			(show_name no)
@@
 			)
 		)
-		(property "Value" "2.2u"
+		(property "Value" "2.2uF"
 			(at 156.464 120.396 0)
 			(show_name no)
@@
 			)
 		)
-		(property "Value" "47n"
+		(property "Value" "47nF"
 			(at 209.55 115.5762 0)
 			(show_name no)
@@
 			)
 		)
-		(property "Value" "2.2u"
+		(property "Value" "2.2uF"
 			(at 125.984 110.236 0)
 			(show_name no)
@@
 			)
 		)
-		(property "Manufacturer" ""
-			(at 184.15 123.19 0)
-			(hide yes)
-			(show_name no)
-			(do_not_autoplace no)
-			(effects
-				(font
-					(size 1.27 1.27)
-				)
-			)
-		)
 		(property "Manufacturer Part Number" ""
 			(at 184.15 123.19 0)
@@
 		)
 		(property "FT Origin" ""
+			(at 184.15 123.19 0)
+			(hide yes)
+			(show_name no)
+			(do_not_autoplace no)
+			(effects
+				(font
+					(size 1.27 1.27)
+				)
+			)
+		)
+		(property "*LCSC Part Number" "C2842775"
 			(at 184.15 123.19 0)
 			(hide yes)
@@
 			)
 		)
-		(property "Value" "10u"
+		(property "Value" "10uF"
 			(at 137.414 115.316 0)
 			(show_name no)

Commit message: first Claude Software
Parts:
- BT1: LCSC Part # (none) -> C122425
- C1, C5: LCSC Part # (none) -> C23630
- C2, C3: LCSC Part # (none) -> C13585
- C4: LCSC Part # (none) -> C1622
- D1: LCSC Part # (none) -> C2286
- J1: LCSC Part # (none) -> C160388
- L1: value 2.2u -> 2.2uH; LCSC Part # (none) -> C2847475
- R1, R5: LCSC Part # (none) -> C25804
- R2: LCSC Part # (none) -> C23158
- R3: LCSC Part # (none) -> C137769
- R4: *LCSC Part Number C21189 -> C22765; LCSC Part # (none) -> C22765
- R6: LCSC Part # (none) -> C21189
- U1: LCSC Part # (none) -> C2842775
Changed lines of the file:
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@@
+			)
+		)
+		(property "LCSC Part #" "C122425"
+			(at 236.22 129.54 0)
+			(hide yes)
+			(show_name no)
+			(do_not_autoplace no)
+			(effects
+				(font
+					(size 1.27 1.27)
+				)
 			)
 		)
@@
 			)
 		)
+		(property "LCSC Part #" "C25804"
+			(at 160.02 138.43 90)
+			(hide yes)
+			(show_name no)
+			(do_not_autoplace no)
+			(effects
+				(font
+					(size 1.27 1.27)
+				)
+			)
+		)
 		(pin "1"
 		)
@@
 			)
 		)
+		(property "LCSC Part #" "C13585"
+			(at 223.52 113.03 0)
+			(hide yes)
+			(show_name no)
+			(do_not_autoplace no)
+			(effects
+				(font
+					(size 1.27 1.27)
+				)
+			)
+		)
 		(pin "2"
 		)
@@
 		)
 		(property "*LCSC Part Number" "C2286"
+			(at 158.75 133.35 0)
+			(hide yes)
+			(show_name no)
+			(do_not_autoplace no)
+			(effects
+				(font
+					(size 1.27 1.27)
+				)
+			)
+		)
+		(property "LCSC Part #" "C2286"
 			(at 158.75 133.35 0)
 			(hide yes)
@@
 			)
 		)
+		(property "LCSC Part #" "C23158"
+			(at 279.4 114.3 0)
+			(hide yes)
+			(show_name no)
+			(do_not_autoplace no)
+			(effects
+				(font
+					(size 1.27 1.27)
+				)
+			)
+		)
 		(pin "1"
 		)
@@
 			)
 		)
+		(property "LCSC Part #" "C21189"
+			(at 160.02 143.51 90)
+			(hide yes)
+			(show_name no)
+			(do_not_autoplace no)
+			(effects
+				(font
+					(size 1.27 1.27)
+				)
+			)
+		)
 		(pin "1"
 		)
@@
 			)
 		)
+		(property "LCSC Part #" "C23630"
+			(at 162.56 119.38 0)
+			(hide yes)
+			(show_name no)
+			(do_not_autoplace no)
+			(effects
+				(font
+					(size 1.27 1.27)
+				)
+			)
+		)
 		(pin "2"
 		)
@@
 			)
 		)
+		(property "LCSC Part #" "C1622"
+			(at 207.01 114.3 0)
+			(hide yes)
+			(show_name no)
+			(do_not_autoplace no)
+			(effects
+				(font
+					(size 1.27 1.27)
+				)
+			)
+		)
 		(pin "1"
 		)
@@
 		)
 		(property "*LCSC Part Number" "C23630"
+			(at 132.08 109.22 0)
+			(hide yes)
+			(show_name no)
+			(do_not_autoplace no)
+			(effects
+				(font
+					(size 1.27 1.27)
+				)
+			)
+		)
+		(property "LCSC Part #" "C23630"
 			(at 132.08 109.22 0)
 			(hide yes)
@@
 			)
 		)
+		(property "LCSC Part #" "C160388"
+			(at 298.45 123.19 0)
+			(hide yes)
+			(show_name no)
+			(do_not_autoplace no)
+			(effects
+				(font
+					(size 1.27 1.27)
+				)
+			)
+		)
 		(pin "2"
 		)
@@
 			)
 		)
-		(property "Value" "2.2u"
+		(property "Value" "2.2uH"
 			(at 214.63 106.68 90)
 			(show_name no)
@@
 		(property "*Distributor Part Number" ""
 			(at 214.63 109.22 0)
+			(hide yes)
+			(show_name no)
+			(do_not_autoplace no)
+			(effects
+				(font
+					(size 1.27 1.27)
+				)
+			)
+		)
+		(property "LCSC Part #" "C2847475"
+			(at 214.63 109.22 90)
 			(hide yes)
 			(show_name no)
@@
 			)
 		)
-		(property "*LCSC Part Number" "C21189"
+		(property "*LCSC Part Number" "C22765"
 			(at 151.13 133.35 0)
+			(hide yes)
+			(show_name no)
+			(do_not_autoplace no)
+			(effects
+				(font
+					(size 1.27 1.27)
+				)
+			)
+		)
+		(property "LCSC Part #" "C22765"
+			(at 151.13 133.35 90)
 			(hide yes)
 			(show_name no)
@@
 			)
 		)
+		(property "LCSC Part #" "C137769"
+			(at 279.4 124.46 0)
+			(hide yes)
+			(show_name no)
+			(do_not_autoplace no)
+			(effects
+				(font
+					(size 1.27 1.27)
+				)
+			)
+		)
 		(pin "1"
 		)
@@
 			)
 		)
-		(property "LCSC Part #" ""
+		(property "LCSC Part #" "C2842775"
 			(at 184.15 123.19 0)
 			(hide yes)
@@
 		)
 		(property "*LCSC Part Number" "C13585"
+			(at 143.51 114.3 0)
+			(hide yes)
+			(show_name no)
+			(do_not_autoplace no)
+			(effects
+				(font
+					(size 1.27 1.27)
+				)
+			)
+		)
+		(property "LCSC Part #" "C13585"
 			(at 143.51 114.3 0)
 			(hide yes)
@@
 			(at 158.75 104.14 0)
 			(hide yes)
+			(show_name no)
+			(do_not_autoplace no)
+			(effects
+				(font
+					(size 1.27 1.27)
+				)
+			)
+		)
+		(property "LCSC Part #" "C25804"
+			(at 158.75 104.14 0)
+			(hide yes)
