File: Hardware/Electrical/PCB_v2/PCB_v2.kicad_pcb (KiCad board)
At the start: 6 copper layers, 1 part

Commit message: manual LED circle done
Parts:
- removed REF**: IC_LM73100RPWR, LM73100:IC_LM73100RPWR
- added BT1: Battery_Cell, Connector_Molex:Molex_Micro-Fit_3.0_43650-0224_1x02-1MP_P3.00mm_Vertical, F.Cu at (36.4, 71.4)
- added C1: 2.2u, Capacitor_SMD:C_0603_1608Metric, F.Cu at (26.3, 69.5)
- added C10: 0.1 uF, Capacitor_SMD:C_0603_1608Metric, F.Cu at (34.8, 51.3)
- added C100: 1u, Capacitor_SMD:C_0603_1608Metric, F.Cu at (408.1, 135.3)
- added C101: 1u, Capacitor_SMD:C_0603_1608Metric, F.Cu at (376.1, 143.3)
- added C102: 1u, Capacitor_SMD:C_0603_1608Metric, F.Cu at (384.1, 143.3)
- added C103: 1u, Capacitor_SMD:C_0603_1608Metric, F.Cu at (392.1, 143.3)
- added C11: 1uF, Capacitor_SMD:C_0603_1608Metric, F.Cu at (34.8, 53.8)
- added C12: 1uF, Capacitor_SMD:C_0603_1608Metric, F.Cu at (38.8, 41.3)
- added C13: 0.1 uF, Capacitor_SMD:C_0603_1608Metric, F.Cu at (38.8, 43.8)
- added C14: 0.1 uF, Capacitor_SMD:C_0603_1608Metric, F.Cu at (38.8, 46.3)
- added C15: 100n, Capacitor_SMD:C_0603_1608Metric, F.Cu at (12.2, 109.5)
- added C16: 22u, Capacitor_SMD:C_1206_3216Metric, F.Cu at (7.38, 109.9)
- added C17: 1u, Capacitor_SMD:C_0603_1608Metric, F.Cu at (12.2, 112.0)
- added C18: 100n, Capacitor_SMD:C_0603_1608Metric, F.Cu at (12.2, 114.5)
- added C19: 22u, Capacitor_SMD:C_1206_3216Metric, F.Cu at (7.38, 113.2)
- added C2: 10u, Capacitor_SMD:C_1206_3216Metric, F.Cu at (39.2, 78.5)
- added C20: 22u, Capacitor_SMD:C_1206_3216Metric, F.Cu at (7.38, 116.6)
- added C21: 22u, Capacitor_SMD:C_1206_3216Metric, F.Cu at (7.38, 119.9)
- added C22: 1u, Capacitor_SMD:C_0603_1608Metric, F.Cu at (12.2, 117.0)
- added C23: 100n, Capacitor_SMD:C_0603_1608Metric, F.Cu at (12.2, 119.5)
- added C24: 22p, Capacitor_SMD:C_0603_1608Metric, F.Cu at (12.2, 122.0)
- added C25: x, Capacitor_SMD:C_0603_1608Metric, F.Cu at (12.2, 124.5)
- added C26: 1u, Capacitor_SMD:C_0603_1608Metric, F.Cu at (12.2, 127.0)
- added C27: 22u, Capacitor_SMD:C_1206_3216Metric, F.Cu at (7.38, 123.3)
- added C28: 1u, Capacitor_SMD:C_0603_1608Metric, F.Cu at (12.2, 129.5)
- added C29: 100n, Capacitor_SMD:C_0603_1608Metric, F.Cu at (12.2, 132.0)
- added C3: 10u, Capacitor_SMD:C_1206_3216Metric, F.Cu at (39.2, 81.9)
- added C30: 22u, Capacitor_SMD:C_1206_3216Metric, F.Cu at (7.38, 126.6)
- added C31: 22u, Capacitor_SMD:C_1206_3216Metric, F.Cu at (7.38, 130.0)
- added C32: 22u, Capacitor_SMD:C_1206_3216Metric, F.Cu at (7.38, 133.3)
- added C33: 1u, Capacitor_SMD:C_0603_1608Metric, F.Cu at (16.2, 109.5)
- added C34: 100n, Capacitor_SMD:C_0603_1608Metric, F.Cu at (16.2, 112.0)
- added C35: 1u, Capacitor_SMD:C_0603_1608Metric, F.Cu at (16.2, 114.5)
- added C36: 1u, Capacitor_SMD:C_0603_1608Metric, F.Cu at (16.2, 117.0)
- added C37: 100n, Capacitor_SMD:C_0603_1608Metric, F.Cu at (16.2, 119.5)
- added C38: 2.2u, Capacitor_SMD:C_0603_1608Metric, F.Cu at (16.2, 122.0)
- added C39: 2.2u, Capacitor_SMD:C_0603_1608Metric, F.Cu at (16.2, 124.5)
- added C4: 47n, Capacitor_SMD:C_0603_1608Metric, F.Cu at (26.3, 72.0)
- added C40: 100n, Capacitor_SMD:C_0603_1608Metric, F.Cu at (16.2, 127.0)
- added C41: 10u, Capacitor_SMD:C_1206_3216Metric, F.Cu at (7.38, 136.7)
- added C42: 2.2u, Capacitor_SMD:C_0603_1608Metric, F.Cu at (16.2, 129.5)
- added C43: 100n, Capacitor_SMD:C_0603_1608Metric, F.Cu at (16.2, 132.0)
- added C44: 1u, Capacitor_SMD:C_0603_1608Metric, F.Cu at (376.1, 79.3)
- added C45: 1u, Capacitor_SMD:C_0603_1608Metric, F.Cu at (384.1, 79.3)
- added C46: 1u, Capacitor_SMD:C_0603_1608Metric, F.Cu at (392.1, 79.3)
- added C47: 1u, Capacitor_SMD:C_0603_1608Metric, F.Cu at (360.1, 87.3)
- added C48: 1u, Capacitor_SMD:C_0603_1608Metric, F.Cu at (368.1, 87.3)
- added C49: 1u, Capacitor_SMD:C_0603_1608Metric, F.Cu at (376.1, 87.3)
- added C5: 2.2u, Capacitor_SMD:C_0603_1608Metric, F.Cu at (26.3, 74.5)
- added C50: 1u, Capacitor_SMD:C_0603_1608Metric, F.Cu at (384.1, 87.3)
- added C51: 1u, Capacitor_SMD:C_0603_1608Metric, F.Cu at (392.1, 87.3)
- added C52: 1u, Capacitor_SMD:C_0603_1608Metric, F.Cu at (400.1, 87.3)
- added C53: 1u, Capacitor_SMD:C_0603_1608Metric, F.Cu at (408.1, 87.3)
- added C54: 1u, Capacitor_SMD:C_0603_1608Metric, F.Cu at (360.1, 95.3)
- added C55: 1u, Capacitor_SMD:C_0603_1608Metric, F.Cu at (368.1, 95.3)
- added C56: 1u, Capacitor_SMD:C_0603_1608Metric, F.Cu at (376.1, 95.3)
- added C57: 1u, Capacitor_SMD:C_0603_1608Metric, F.Cu at (384.1, 95.3)
- added C58: 1u, Capacitor_SMD:C_0603_1608Metric, F.Cu at (392.1, 95.3)
- added C59: 1u, Capacitor_SMD:C_0603_1608Metric, F.Cu at (400.1, 95.3)
- added C6: 1uF, Capacitor_SMD:C_0603_1608Metric, F.Cu at (34.8, 41.3)
- added C60: 1u, Capacitor_SMD:C_0603_1608Metric, F.Cu at (408.6, 95.3)
- added C61: 1u, Capacitor_SMD:C_0603_1608Metric, F.Cu at (352.1, 103.3)
- added C62: 1u, Capacitor_SMD:C_0603_1608Metric, F.Cu at (360.1, 103.3)
- added C63: 1u, Capacitor_SMD:C_0603_1608Metric, F.Cu at (368.1, 103.3)
- added C64: 1u, Capacitor_SMD:C_0603_1608Metric, F.Cu at (376.1, 103.3)
- added C65: 1u, Capacitor_SMD:C_0603_1608Metric, F.Cu at (384.1, 103.3)
- added C66: 1u, Capacitor_SMD:C_0603_1608Metric, F.Cu at (392.1, 103.3)
- added C67: 1u, Capacitor_SMD:C_0603_1608Metric, F.Cu at (400.1, 103.3)
- added C68: 1u, Capacitor_SMD:C_0603_1608Metric, F.Cu at (408.1, 103.3)
- added C69: 1u, Capacitor_SMD:C_0603_1608Metric, F.Cu at (416.1, 103.3)
- added C7: 1uF, Capacitor_SMD:C_0603_1608Metric, F.Cu at (34.8, 43.8)
- added C70: 1u, Capacitor_SMD:C_0603_1608Metric, F.Cu at (352.1, 111.3)
- added C71: 1u, Capacitor_SMD:C_0603_1608Metric, F.Cu at (360.1, 111.3)
- added C72: 1u, Capacitor_SMD:C_0603_1608Metric, F.Cu at (368.1, 111.3)
- added C73: 1u, Capacitor_SMD:C_0603_1608Metric, F.Cu at (376.1, 111.3)
- added C74: 1u, Capacitor_SMD:C_0603_1608Metric, F.Cu at (392.1, 111.3)
- added C75: 1u, Capacitor_SMD:C_0603_1608Metric, F.Cu at (400.1, 111.3)
- added C76: 1u, Capacitor_SMD:C_0603_1608Metric, F.Cu at (408.1, 111.3)
- added C77: 1u, Capacitor_SMD:C_0603_1608Metric, F.Cu at (416.1, 111.3)
- added C78: 1u, Capacitor_SMD:C_0603_1608Metric, F.Cu at (352.1, 119.3)
- added C79: 1u, Capacitor_SMD:C_0603_1608Metric, F.Cu at (360.1, 119.3)
- added C8: 0.1 uF, Capacitor_SMD:C_0603_1608Metric, F.Cu at (34.8, 46.3)
- added C80: 1u, Capacitor_SMD:C_0603_1608Metric, F.Cu at (368.1, 119.3)
- added C81: 1u, Capacitor_SMD:C_0603_1608Metric, F.Cu at (376.1, 119.3)
- added C82: 1u, Capacitor_SMD:C_0603_1608Metric, F.Cu at (384.1, 119.3)
- added C83: 1u, Capacitor_SMD:C_0603_1608Metric, F.Cu at (392.1, 119.3)
- added C84: 1u, Capacitor_SMD:C_0603_1608Metric, F.Cu at (400.1, 119.3)
- added C85: 1u, Capacitor_SMD:C_0603_1608Metric, F.Cu at (408.1, 119.3)
- added C86: 1u, Capacitor_SMD:C_0603_1608Metric, F.Cu at (416.1, 119.3)
- added C87: 1u, Capacitor_SMD:C_0603_1608Metric, F.Cu at (360.1, 127.3)
- added C88: 1u, Capacitor_SMD:C_0603_1608Metric, F.Cu at (368.1, 127.3)
- added C89: 1u, Capacitor_SMD:C_0603_1608Metric, F.Cu at (376.1, 127.3)
- added C9: 0.1 uF, Capacitor_SMD:C_0603_1608Metric, F.Cu at (34.8, 48.8)
- added C90: 1u, Capacitor_SMD:C_0603_1608Metric, F.Cu at (384.1, 127.3)
- added C91: 1u, Capacitor_SMD:C_0603_1608Metric, F.Cu at (392.1, 127.3)
- added C92: 1u, Capacitor_SMD:C_0603_1608Metric, F.Cu at (400.1, 127.3)
- added C93: 1u, Capacitor_SMD:C_0603_1608Metric, F.Cu at (408.1, 127.3)
- added C94: 1u, Capacitor_SMD:C_0603_1608Metric, F.Cu at (360.1, 135.3)
- added C95: 1u, Capacitor_SMD:C_0603_1608Metric, F.Cu at (368.1, 135.3)
- added C96: 1u, Capacitor_SMD:C_0603_1608Metric, F.Cu at (376.1, 135.3)
- added C97: 1u, Capacitor_SMD:C_0603_1608Metric, F.Cu at (384.1, 135.3)
- added C98: 1u, Capacitor_SMD:C_0603_1608Metric, F.Cu at (392.1, 135.3)
- added C99: 1u, Capacitor_SMD:C_0603_1608Metric, F.Cu at (400.1, 135.3)
- added D1: Orange, LED_SMD:LED_0603_1608Metric, F.Cu at (44.0, 78.1)
- added D10: WS2812B, LED_SMD:LED_WS2812B_PLCC4_5.0x5.0mm_P3.2mm, F.Cu at (384.0, 83.5)
- added D11: WS2812B, LED_SMD:LED_WS2812B_PLCC4_5.0x5.0mm_P3.2mm, F.Cu at (392.0, 83.5)
- added D12: WS2812B, LED_SMD:LED_WS2812B_PLCC4_5.0x5.0mm_P3.2mm, F.Cu at (400.0, 83.5)
- added D13: WS2812B, LED_SMD:LED_WS2812B_PLCC4_5.0x5.0mm_P3.2mm, F.Cu at (408.0, 83.5)
- added D14: WS2812B, LED_SMD:LED_WS2812B_PLCC4_5.0x5.0mm_P3.2mm, F.Cu at (360.0, 91.5)
- added D15: WS2812B, LED_SMD:LED_WS2812B_PLCC4_5.0x5.0mm_P3.2mm, F.Cu at (368.0, 91.5)
- added D16: WS2812B, LED_SMD:LED_WS2812B_PLCC4_5.0x5.0mm_P3.2mm, F.Cu at (376.0, 91.5)
- added D17: WS2812B, LED_SMD:LED_WS2812B_PLCC4_5.0x5.0mm_P3.2mm, F.Cu at (384.0, 91.5)
- added D18: WS2812B, LED_SMD:LED_WS2812B_PLCC4_5.0x5.0mm_P3.2mm, F.Cu at (392.0, 91.5)
- added D19: WS2812B, LED_SMD:LED_WS2812B_PLCC4_5.0x5.0mm_P3.2mm, F.Cu at (400.0, 91.5)
- added D20: WS2812B, LED_SMD:LED_WS2812B_PLCC4_5.0x5.0mm_P3.2mm, F.Cu at (408.5, 91.5)
- added D21: WS2812B, LED_SMD:LED_WS2812B_PLCC4_5.0x5.0mm_P3.2mm, F.Cu at (352.0, 99.5)
- added D22: WS2812B, LED_SMD:LED_WS2812B_PLCC4_5.0x5.0mm_P3.2mm, F.Cu at (360.0, 99.5)
- added D23: WS2812B, LED_SMD:LED_WS2812B_PLCC4_5.0x5.0mm_P3.2mm, F.Cu at (368.0, 99.5)
- added D24: WS2812B, LED_SMD:LED_WS2812B_PLCC4_5.0x5.0mm_P3.2mm, F.Cu at (376.0, 99.5)
- added D25: WS2812B, LED_SMD:LED_WS2812B_PLCC4_5.0x5.0mm_P3.2mm, F.Cu at (384.0, 99.5)
- added D26: WS2812B, LED_SMD:LED_WS2812B_PLCC4_5.0x5.0mm_P3.2mm, F.Cu at (392.0, 99.5)
- added D27: WS2812B, LED_SMD:LED_WS2812B_PLCC4_5.0x5.0mm_P3.2mm, F.Cu at (400.0, 99.5)
- added D28: WS2812B, LED_SMD:LED_WS2812B_PLCC4_5.0x5.0mm_P3.2mm, F.Cu at (408.0, 99.5)
- added D29: WS2812B, LED_SMD:LED_WS2812B_PLCC4_5.0x5.0mm_P3.2mm, F.Cu at (416.0, 99.5)
- added D30: WS2812B, LED_SMD:LED_WS2812B_PLCC4_5.0x5.0mm_P3.2mm, F.Cu at (352.0, 107.5)
- added D31: WS2812B, LED_SMD:LED_WS2812B_PLCC4_5.0x5.0mm_P3.2mm, F.Cu at (360.0, 107.5)
- added D32: WS2812B, LED_SMD:LED_WS2812B_PLCC4_5.0x5.0mm_P3.2mm, F.Cu at (368.0, 107.5)
- added D33: WS2812B, LED_SMD:LED_WS2812B_PLCC4_5.0x5.0mm_P3.2mm, F.Cu at (376.0, 107.5)
- added D34: WS2812B, LED_SMD:LED_WS2812B_PLCC4_5.0x5.0mm_P3.2mm, F.Cu at (392.0, 107.5)
- added D35: WS2812B, LED_SMD:LED_WS2812B_PLCC4_5.0x5.0mm_P3.2mm, F.Cu at (400.0, 107.5)
- added D36: WS2812B, LED_SMD:LED_WS2812B_PLCC4_5.0x5.0mm_P3.2mm, F.Cu at (408.0, 107.5)
- added D37: WS2812B, LED_SMD:LED_WS2812B_PLCC4_5.0x5.0mm_P3.2mm, F.Cu at (416.0, 107.5)
- added D38: WS2812B, LED_SMD:LED_WS2812B_PLCC4_5.0x5.0mm_P3.2mm, F.Cu at (352.0, 115.5)
- added D39: WS2812B, LED_SMD:LED_WS2812B_PLCC4_5.0x5.0mm_P3.2mm, F.Cu at (360.0, 115.5)
- added D4: WS2812B, LED_SMD:LED_WS2812B_PLCC4_5.0x5.0mm_P3.2mm, F.Cu at (376.0, 75.5)
- added D40: WS2812B, LED_SMD:LED_WS2812B_PLCC4_5.0x5.0mm_P3.2mm, F.Cu at (368.0, 115.5)
- added D41: WS2812B, LED_SMD:LED_WS2812B_PLCC4_5.0x5.0mm_P3.2mm, F.Cu at (376.0, 115.5)
- added D42: WS2812B, LED_SMD:LED_WS2812B_PLCC4_5.0x5.0mm_P3.2mm, F.Cu at (384.0, 115.5)
- added D43: WS2812B, LED_SMD:LED_WS2812B_PLCC4_5.0x5.0mm_P3.2mm, F.Cu at (392.0, 115.5)
- added D44: WS2812B, LED_SMD:LED_WS2812B_PLCC4_5.0x5.0mm_P3.2mm, F.Cu at (400.0, 115.5)
- added D45: WS2812B, LED_SMD:LED_WS2812B_PLCC4_5.0x5.0mm_P3.2mm, F.Cu at (408.0, 115.5)
- added D46: WS2812B, LED_SMD:LED_WS2812B_PLCC4_5.0x5.0mm_P3.2mm, F.Cu at (416.0, 115.5)
- added D47: WS2812B, LED_SMD:LED_WS2812B_PLCC4_5.0x5.0mm_P3.2mm, F.Cu at (360.0, 123.5)
- added D48: WS2812B, LED_SMD:LED_WS2812B_PLCC4_5.0x5.0mm_P3.2mm, F.Cu at (368.0, 123.5)
- added D49: WS2812B, LED_SMD:LED_WS2812B_PLCC4_5.0x5.0mm_P3.2mm, F.Cu at (376.0, 123.5)
- added D5: WS2812B, LED_SMD:LED_WS2812B_PLCC4_5.0x5.0mm_P3.2mm, F.Cu at (384.0, 75.5)
- added D50: WS2812B, LED_SMD:LED_WS2812B_PLCC4_5.0x5.0mm_P3.2mm, F.Cu at (384.0, 123.5)
- added D51: WS2812B, LED_SMD:LED_WS2812B_PLCC4_5.0x5.0mm_P3.2mm, F.Cu at (392.0, 123.5)
- added D52: WS2812B, LED_SMD:LED_WS2812B_PLCC4_5.0x5.0mm_P3.2mm, F.Cu at (400.0, 123.5)
- added D53: WS2812B, LED_SMD:LED_WS2812B_PLCC4_5.0x5.0mm_P3.2mm, F.Cu at (408.0, 123.5)
- added D54: WS2812B, LED_SMD:LED_WS2812B_PLCC4_5.0x5.0mm_P3.2mm, F.Cu at (360.0, 131.5)
- added D55: WS2812B, LED_SMD:LED_WS2812B_PLCC4_5.0x5.0mm_P3.2mm, F.Cu at (368.0, 131.5)
- added D56: WS2812B, LED_SMD:LED_WS2812B_PLCC4_5.0x5.0mm_P3.2mm, F.Cu at (376.0, 131.5)
- added D57: WS2812B, LED_SMD:LED_WS2812B_PLCC4_5.0x5.0mm_P3.2mm, F.Cu at (384.0, 131.5)
- added D58: WS2812B, LED_SMD:LED_WS2812B_PLCC4_5.0x5.0mm_P3.2mm, F.Cu at (392.0, 131.5)
- added D59: WS2812B, LED_SMD:LED_WS2812B_PLCC4_5.0x5.0mm_P3.2mm, F.Cu at (400.0, 131.5)
- added D6: WS2812B, LED_SMD:LED_WS2812B_PLCC4_5.0x5.0mm_P3.2mm, F.Cu at (392.0, 75.5)
- added D60: WS2812B, LED_SMD:LED_WS2812B_PLCC4_5.0x5.0mm_P3.2mm, F.Cu at (408.0, 131.5)
- added D61: WS2812B, LED_SMD:LED_WS2812B_PLCC4_5.0x5.0mm_P3.2mm, F.Cu at (376.0, 139.5)
- added D62: WS2812B, LED_SMD:LED_WS2812B_PLCC4_5.0x5.0mm_P3.2mm, F.Cu at (384.0, 139.5)
- added D63: WS2812B, LED_SMD:LED_WS2812B_PLCC4_5.0x5.0mm_P3.2mm, F.Cu at (392.0, 139.5)
- added D7: WS2812B, LED_SMD:LED_WS2812B_PLCC4_5.0x5.0mm_P3.2mm, F.Cu at (360.0, 83.5)
- added D8: WS2812B, LED_SMD:LED_WS2812B_PLCC4_5.0x5.0mm_P3.2mm, F.Cu at (368.0, 83.5)
- added D9: WS2812B, LED_SMD:LED_WS2812B_PLCC4_5.0x5.0mm_P3.2mm, F.Cu at (376.0, 83.5)
- added J1: 10k NTC, Connector_JST:JST_SH_BM02B-SRSS-TB_1x02-1MP_P1.00mm_Vertical, F.Cu at (31.7, 86.7)
- added J2: USB_C_Receptacle_USB2.0_16P, Connector_USB:USB_C_Receptacle_GCT_USB4105-xx-A_16P_TopMnt_Horizontal, F.Cu at (38.7, 60.3)
- added J3: 1, Connector_JST:JST_XH_B1B-XH-AM_1x01_P2.50mm_Vertical, F.Cu at (-47.0, 153.8)
- added J4: 1, Connector_JST:JST_XH_B1B-XH-AM_1x01_P2.50mm_Vertical, F.Cu at (-40.1, 153.8)
- added J5: 1, Connector_JST:JST_XH_B1B-XH-AM_1x01_P2.50mm_Vertical, F.Cu at (-33.1, 153.8)
- added J6: 1, Connector_JST:JST_XH_B1B-XH-AM_1x01_P2.50mm_Vertical, F.Cu at (-26.2, 153.8)
- added J7: 1, Connector_JST:JST_XH_B1B-XH-AM_1x01_P2.50mm_Vertical, F.Cu at (-19.2, 153.8)
- added J8: 1, Connector_JST:JST_XH_B1B-XH-AM_1x01_P2.50mm_Vertical, F.Cu at (-12.3, 153.8)
- added L1: 2.2u, Inductor_SMD:L_Bourns_SRP5030T, F.Cu at (32.3, 80.2)
- added L2: 1uH, Inductor_SMD:L_Bourns_SRP7028A_7.3x6.6mm, F.Cu at (35.2, 112.3)
- added L3: 1uH, Inductor_SMD:L_Bourns_SRP7028A_7.3x6.6mm, F.Cu at (35.2, 120.4)
- added L4: 4.7uH, Inductor_SMD:L_Pulse_PA5402, F.Cu at (18.4, 136.1)
- added Q1: Q_PMOS, 0_CRS_lib:PowerPAK_SO-8, F.Cu at (26.1, 41.4)
- added Q2: Q_PMOS, 0_CRS_lib:PowerPAK_SO-8, F.Cu at (26.1, 47.9)
- added Q3: Q_PMOS, 0_CRS_lib:PowerPAK_SO-8, F.Cu at (26.1, 54.5)
- added Q4: Q_PMOS, 0_CRS_lib:PowerPAK_SO-8, F.Cu at (26.1, 61.0)
- added R1: 10k, Resistor_SMD:R_0603_1608Metric, F.Cu at (26.3, 77.0)
- added R11: 1k, Resistor_SMD:R_0603_1608Metric, F.Cu at (38.8, 53.8)
- added R12: 1k, Resistor_SMD:R_0603_1608Metric, F.Cu at (42.8, 41.3)
- added R14: 0 Ohm, Resistor_SMD:R_0603_1608Metric, F.Cu at (42.8, 43.8)
- added R15: 0 Ohm, Resistor_SMD:R_0603_1608Metric, F.Cu at (42.8, 46.3)
- added R16: 0 Ohm, Resistor_SMD:R_0603_1608Metric, F.Cu at (42.8, 48.8)
- added R17: 0 Ohm, Resistor_SMD:R_0603_1608Metric, F.Cu at (42.8, 51.3)
- added R18: 51k, Resistor_SMD:R_0603_1608Metric, F.Cu at (20.2, 109.5)
- added R19: 51, Resistor_SMD:R_0603_1608Metric, F.Cu at (20.2, 112.0)
- added R2: 4.32k, Resistor_SMD:R_0603_1608Metric, F.Cu at (26.3, 79.5)
- added R20: 240k, Resistor_SMD:R_0603_1608Metric, F.Cu at (20.2, 114.5)
- added R21: 750k, Resistor_SMD:R_0603_1608Metric, F.Cu at (20.2, 117.0)
- added R22: 150k, Resistor_SMD:R_0603_1608Metric, F.Cu at (20.2, 119.5)
- added R23: 62k, Resistor_SMD:R_0603_1608Metric, F.Cu at (20.2, 122.0)
- added R24: 300k, Resistor_SMD:R_0603_1608Metric, F.Cu at (20.2, 124.5)
- added R25: 91k, Resistor_SMD:R_0603_1608Metric, F.Cu at (20.2, 127.0)
- added R26: 100k, Resistor_SMD:R_0603_1608Metric, F.Cu at (20.2, 129.5)
- added R27: 20k, Resistor_SMD:R_0603_1608Metric, F.Cu at (20.2, 132.0)
- added R28: 100k, Resistor_SMD:R_0603_1608Metric, F.Cu at (24.2, 109.5)
- added R29: 0, Resistor_SMD:R_0603_1608Metric, F.Cu at (24.2, 112.0)
- added R3: 21k, Resistor_SMD:R_0603_1608Metric, F.Cu at (26.3, 82.0)
- added R30: 91k, Resistor_SMD:R_0603_1608Metric, F.Cu at (24.2, 114.5)
- added R31: 750k, Resistor_SMD:R_0603_1608Metric, F.Cu at (24.2, 117.0)
- added R32: 91k, Resistor_SMD:R_0603_1608Metric, F.Cu at (24.2, 119.5)
- added R33: 732k, Resistor_SMD:R_0603_1608Metric, F.Cu at (24.2, 122.0)
- added R34: 240k, Resistor_SMD:R_0603_1608Metric, F.Cu at (24.2, 124.5)
- added R35: 100k, Resistor_SMD:R_0603_1608Metric, F.Cu at (24.2, 127.0)
- added R36: 62k, Resistor_SMD:R_0603_1608Metric, F.Cu at (24.2, 129.5)
- added R37: 300k, Resistor_SMD:R_0603_1608Metric, F.Cu at (24.2, 132.0)
- added R38: 100k, Resistor_SMD:R_0603_1608Metric, F.Cu at (28.3, 109.5)
- added R39: 91k, Resistor_SMD:R_0603_1608Metric, F.Cu at (28.3, 112.0)
- added R4: 120, Resistor_SMD:R_0603_1608Metric, F.Cu at (26.3, 84.5)
- added R40: 10k, Resistor_SMD:R_0603_1608Metric, F.Cu at (28.3, 114.5)
- added R41: 10k, Resistor_SMD:R_0603_1608Metric, F.Cu at (28.3, 117.0)
- added R42: 115k, Resistor_SMD:R_0603_1608Metric, F.Cu at (28.3, 119.5)
- added R43: 49.9k, Resistor_SMD:R_0603_1608Metric, F.Cu at (28.3, 122.0)
- added R44: 10k, Resistor_SMD:R_0603_1608Metric, F.Cu at (0.56, 109.5)
- added R45: 4.7k, Resistor_SMD:R_0603_1608Metric, F.Cu at (0.56, 112.0)
- added R46: 4.7k, Resistor_SMD:R_0603_1608Metric, F.Cu at (0.56, 114.5)
- added R47: 4.7k, Resistor_SMD:R_0603_1608Metric, F.Cu at (0.56, 117.0)
- added R48: 10k, Resistor_SMD:R_0603_1608Metric, F.Cu at (0.56, 119.5)
- added R49: 100, Resistor_SMD:R_0603_1608Metric, F.Cu at (295.4, 138.1)
- added R5: 10k, Resistor_SMD:R_0603_1608Metric, F.Cu at (26.3, 87.0)
- added R50: 0, Resistor_SMD:R_0603_1608Metric, F.Cu at (20.3, 56.3)
- added R51: 4.7k, Resistor_SMD:R_0603_1608Metric, F.Cu at (20.3, 58.8)
- added R52: 0, Resistor_SMD:R_0603_1608Metric, F.Cu at (20.3, 61.3)
- added R6: 0, Resistor_SMD:R_0603_1608Metric, F.Cu at (26.3, 89.5)
- added R7: 10k, Resistor_SMD:R_0603_1608Metric, F.Cu at (38.8, 48.8)
- added R9: 2.2k, Resistor_SMD:R_0603_1608Metric, F.Cu at (38.8, 51.3)
- added U1: BQ25303JRTER, Package_DFN_QFN:WQFN-16-1EP_3x3mm_P0.5mm_EP1.68x1.68mm, F.Cu at (39.4, 86.2)
- added U10: ESP32-S3-WROOM-1-N16, RF_Module:ESP32-S3-WROOM-1, F.Cu at (-26.0, 136.5)
- added U11: CAP1296-1-AIA-TR, Package_DFN_QFN:DFN-10-1EP_3x3mm_P0.5mm_EP1.55x2.48mm, F.Cu at (-5.70, 152.8)
- added U12: SN74LVC1T45DRL, Package_TO_SOT_SMD:SOT-563, F.Cu at (-7.08, 156.9)
- added U13: TMP1075DSG, Package_SON:WSON-8-1EP_2x2mm_P0.5mm_EP0.9x1.6mm, F.Cu at (0.43, 69.5)
- added U2: TPD2EUSB30, Package_TO_SOT_SMD:Texas_DRT-3, F.Cu at (46.1, 62.6)
- added U3: CYPD3177-24LQ, Package_DFN_QFN:QFN-24-1EP_4x4mm_P0.5mm_EP2.75x2.75mm, F.Cu at (48.0, 58.2)
- added U4: LM73100RPWR, LM73100:IC_LM73100RPWR, F.Cu at (13.1, 135.3)
- added U5: TPS51385, footprints:VREG_TPS51386RJNR, F.Cu at (24.7, 135.8)
- added U6: TPS61022, Package_DFN_QFN:Texas_RWU0007A_VQFN-7_2x2mm_P0.5mm, F.Cu at (32.5, 135.5)
- added U7: LM73100RPWR, LM73100:IC_LM73100RPWR, F.Cu at (13.1, 139.2)
- added U8: TLV77333PDBVR, Package_TO_SOT_SMD:SOT-23-5, F.Cu at (32.8, 126.9)
- added U9: LMR50410, Package_TO_SOT_SMD:SOT-23-6, F.Cu at (32.8, 131.5)
Routing:
- net /Project Architecture/LED/+LED_POWER: track 0.00 -> 169.7 mm
Other:
- board outline added: 147 x 140 mm

Commit message: Components placed
Parts:
- removed C14: 0.1 uF, Capacitor_SMD:C_0603_1608Metric
- added C104: 100nF, Capacitor_SMD:C_0603_1608Metric, F.Cu at (141.1, 28.9)
- added C105: 100nF, Capacitor_SMD:C_0603_1608Metric, F.Cu at (107.0, 80.0)
- added D2: D_Zener, Diode_SMD:D_SOD-323, F.Cu at (205.7, 86.2)
- added D3: D_Schottky, Package_TO_SOT_SMD:SOT-23, F.Cu at (167.9, 121.5)
- added R10: 49.9k, Resistor_SMD:R_0603_1608Metric, F.Cu at (212.1, 94.4)
- added R13: 4.7k, Resistor_SMD:R_0603_1608Metric, F.Cu at (213.8, 85.0)
- added R8: 49.9k, Resistor_SMD:R_0603_1608Metric, F.Cu at (203.1, 92.1)
- C1, C38, C39, C42, C5: value 2.2u -> 2.2uF
- C10, C13, C8, C9: value 0.1 uF -> 100nF
- C100, C101, C102, C103, C17, C22, C26, C28, C33, C35, C36, C44, C45, C46, C47, C48, C49, C50, C51, C52, C53, C54, C55, C56, C57, C58, C59, C60, C61, C62, C63, C64, C65, C66, C67, C68, C69, C70, C71, C72, C73, C74, C75, C76, C77, C78, C79, C80, C81, C82, C83, C84, C85, C86, C87, C88, C89, C90, C91, C92, C93, C94, C95, C96, C97, C98, C99: value 1u -> 1uF
- C15, C18, C23, C29, C34, C40, C43: value 100n -> 100nF
- C16, C19, C20, C21, C27, C30, C31, C32: value 22u -> 22uF
- C2, C3, C41: value 10u -> 10uF
- C4: value 47n -> 47nF
- J2: moved to B.Cu
- R29, R50, R52, R6: value 0 -> 0 Ohm
- moved C60 234.6 mm to (175.0, 72.8)
- moved D20 234.6 mm to (175.0, 69.0)
- moved C100 234.1 mm to (175.1, 112.8)
- moved C101 234.1 mm to (143.1, 120.8)
- moved C102 234.1 mm to (151.1, 120.8)
- moved C103 234.1 mm to (159.1, 120.8)
- moved C44 234.1 mm to (143.1, 56.8)
- moved C45 234.1 mm to (151.1, 56.8)
- moved C46 234.1 mm to (159.1, 56.8)
- moved C47 234.1 mm to (127.1, 64.8)
- moved C48 234.1 mm to (135.1, 64.8)
- moved C49 234.1 mm to (143.1, 64.8)
- moved C50 234.1 mm to (151.1, 64.8)
- moved C51 234.1 mm to (159.1, 64.8)
- moved C52 234.1 mm to (167.1, 64.8)
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Connections:
- C100 pad 2: /Project Architecture/LED/+LED_POWER -> +5V
- C101 pad 2: /Project Architecture/LED/+LED_POWER -> +5V
- C102 pad 2: /Project Architecture/LED/+LED_POWER -> +5V
- C103 pad 2: /Project Architecture/LED/+LED_POWER -> +5V
- C38 pad 1: /Project Architecture/LED/+LED_POWER -> +5V
- C39 pad 1: /Project Architecture/LED/+LED_POWER -> +5V
- C40 pad 1: /Project Architecture/LED/+LED_POWER -> +5V
- C44 pad 2: /Project Architecture/LED/+LED_POWER -> +5V
- C45 pad 2: /Project Architecture/LED/+LED_POWER -> +5V
- C46 pad 2: /Project Architecture/LED/+LED_POWER -> +5V
- C47 pad 2: /Project Architecture/LED/+LED_POWER -> +5V
- C48 pad 2: /Project Architecture/LED/+LED_POWER -> +5V
- C49 pad 2: /Project Architecture/LED/+LED_POWER -> +5V
- C50 pad 2: /Project Architecture/LED/+LED_POWER -> +5V
- C51 pad 2: /Project Architecture/LED/+LED_POWER -> +5V
- C52 pad 2: /Project Architecture/LED/+LED_POWER -> +5V
- C53 pad 2: /Project Architecture/LED/+LED_POWER -> +5V
- C54 pad 2: /Project Architecture/LED/+LED_POWER -> +5V
- C55 pad 2: /Project Architecture/LED/+LED_POWER -> +5V
- C56 pad 2: /Project Architecture/LED/+LED_POWER -> +5V
- C57 pad 2: /Project Architecture/LED/+LED_POWER -> +5V
- C58 pad 2: /Project Architecture/LED/+LED_POWER -> +5V
- C59 pad 2: /Project Architecture/LED/+LED_POWER -> +5V
- C60 pad 2: /Project Architecture/LED/+LED_POWER -> +5V
- C61 pad 2: /Project Architecture/LED/+LED_POWER -> +5V
- C62 pad 2: /Project Architecture/LED/+LED_POWER -> +5V
- C63 pad 2: /Project Architecture/LED/+LED_POWER -> +5V
- C64 pad 2: /Project Architecture/LED/+LED_POWER -> +5V
- C65 pad 2: /Project Architecture/LED/+LED_POWER -> +5V
- C66 pad 2: /Project Architecture/LED/+LED_POWER -> +5V
- C67 pad 2: /Project Architecture/LED/+LED_POWER -> +5V
- C68 pad 2: /Project Architecture/LED/+LED_POWER -> +5V
- C69 pad 2: /Project Architecture/LED/+LED_POWER -> +5V
- C70 pad 2: /Project Architecture/LED/+LED_POWER -> +5V
- C71 pad 2: /Project Architecture/LED/+LED_POWER -> +5V
- C72 pad 2: /Project Architecture/LED/+LED_POWER -> +5V
- C73 pad 2: /Project Architecture/LED/+LED_POWER -> +5V
- C74 pad 2: /Project Architecture/LED/+LED_POWER -> +5V
- C75 pad 2: /Project Architecture/LED/+LED_POWER -> +5V
- C76 pad 2: /Project Architecture/LED/+LED_POWER -> +5V
- C77 pad 2: /Project Architecture/LED/+LED_POWER -> +5V
- C78 pad 2: /Project Architecture/LED/+LED_POWER -> +5V
- C79 pad 2: /Project Architecture/LED/+LED_POWER -> +5V
- C80 pad 2: /Project Architecture/LED/+LED_POWER -> +5V
- C81 pad 2: /Project Architecture/LED/+LED_POWER -> +5V
- C82 pad 2: /Project Architecture/LED/+LED_POWER -> +5V
- C83 pad 2: /Project Architecture/LED/+LED_POWER -> +5V
- C84 pad 2: /Project Architecture/LED/+LED_POWER -> +5V
- C85 pad 2: /Project Architecture/LED/+LED_POWER -> +5V
- C86 pad 2: /Project Architecture/LED/+LED_POWER -> +5V
- C87 pad 2: /Project Architecture/LED/+LED_POWER -> +5V
- C88 pad 2: /Project Architecture/LED/+LED_POWER -> +5V
- C89 pad 2: /Project Architecture/LED/+LED_POWER -> +5V
- C90 pad 2: /Project Architecture/LED/+LED_POWER -> +5V
- C91 pad 2: /Project Architecture/LED/+LED_POWER -> +5V
- C92 pad 2: /Project Architecture/LED/+LED_POWER -> +5V
- C93 pad 2: /Project Architecture/LED/+LED_POWER -> +5V
- C94 pad 2: /Project Architecture/LED/+LED_POWER -> +5V
- C95 pad 2: /Project Architecture/LED/+LED_POWER -> +5V
- C96 pad 2: /Project Architecture/LED/+LED_POWER -> +5V
- C97 pad 2: /Project Architecture/LED/+LED_POWER -> +5V
- C98 pad 2: /Project Architecture/LED/+LED_POWER -> +5V
- C99 pad 2: /Project Architecture/LED/+LED_POWER -> +5V
- D10 pad 1: /Project Architecture/LED/+LED_POWER -> +5V
- D11 pad 1: /Project Architecture/LED/+LED_POWER -> +5V
- D12 pad 1: /Project Architecture/LED/+LED_POWER -> +5V
- D13 pad 1: /Project Architecture/LED/+LED_POWER -> +5V
- D14 pad 1: /Project Architecture/LED/+LED_POWER -> +5V
- D15 pad 1: /Project Architecture/LED/+LED_POWER -> +5V
- D16 pad 1: /Project Architecture/LED/+LED_POWER -> +5V
- D17 pad 1: /Project Architecture/LED/+LED_POWER -> +5V
- D18 pad 1: /Project Architecture/LED/+LED_POWER -> +5V
- D19 pad 1: /Project Architecture/LED/+LED_POWER -> +5V
- D20 pad 1: /Project Architecture/LED/+LED_POWER -> +5V
- D21 pad 1: /Project Architecture/LED/+LED_POWER -> +5V
- D22 pad 1: /Project Architecture/LED/+LED_POWER -> +5V
- D23 pad 1: /Project Architecture/LED/+LED_POWER -> +5V
- D24 pad 1: /Project Architecture/LED/+LED_POWER -> +5V
- D25 pad 1: /Project Architecture/LED/+LED_POWER -> +5V
- D26 pad 1: /Project Architecture/LED/+LED_POWER -> +5V
- D27 pad 1: /Project Architecture/LED/+LED_POWER -> +5V
- D28 pad 1: /Project Architecture/LED/+LED_POWER -> +5V
- D29 pad 1: /Project Architecture/LED/+LED_POWER -> +5V
- D30 pad 1: /Project Architecture/LED/+LED_POWER -> +5V
- D31 pad 1: /Project Architecture/LED/+LED_POWER -> +5V
- D32 pad 1: /Project Architecture/LED/+LED_POWER -> +5V
- D33 pad 1: /Project Architecture/LED/+LED_POWER -> +5V
- D34 pad 1: /Project Architecture/LED/+LED_POWER -> +5V
- D35 pad 1: /Project Architecture/LED/+LED_POWER -> +5V
- D36 pad 1: /Project Architecture/LED/+LED_POWER -> +5V
- D37 pad 1: /Project Architecture/LED/+LED_POWER -> +5V
- D38 pad 1: /Project Architecture/LED/+LED_POWER -> +5V
- D39 pad 1: /Project Architecture/LED/+LED_POWER -> +5V
- D4 pad 1: /Project Architecture/LED/+LED_POWER -> +5V
- D40 pad 1: /Project Architecture/LED/+LED_POWER -> +5V
- D41 pad 1: /Project Architecture/LED/+LED_POWER -> +5V
- D42 pad 1: /Project Architecture/LED/+LED_POWER -> +5V
- D43 pad 1: /Project Architecture/LED/+LED_POWER -> +5V
- D44 pad 1: /Project Architecture/LED/+LED_POWER -> +5V
- D45 pad 1: /Project Architecture/LED/+LED_POWER -> +5V
- D46 pad 1: /Project Architecture/LED/+LED_POWER -> +5V
- D47 pad 1: /Project Architecture/LED/+LED_POWER -> +5V
- D48 pad 1: /Project Architecture/LED/+LED_POWER -> +5V
- D49 pad 1: /Project Architecture/LED/+LED_POWER -> +5V
- D5 pad 1: /Project Architecture/LED/+LED_POWER -> +5V
- D50 pad 1: /Project Architecture/LED/+LED_POWER -> +5V
- D51 pad 1: /Project Architecture/LED/+LED_POWER -> +5V
- D52 pad 1: /Project Architecture/LED/+LED_POWER -> +5V
- D53 pad 1: /Project Architecture/LED/+LED_POWER -> +5V
- D54 pad 1: /Project Architecture/LED/+LED_POWER -> +5V
- D55 pad 1: /Project Architecture/LED/+LED_POWER -> +5V
- D56 pad 1: /Project Architecture/LED/+LED_POWER -> +5V
- D57 pad 1: /Project Architecture/LED/+LED_POWER -> +5V
- D58 pad 1: /Project Architecture/LED/+LED_POWER -> +5V
- D59 pad 1: /Project Architecture/LED/+LED_POWER -> +5V
- D6 pad 1: /Project Architecture/LED/+LED_POWER -> +5V
- D60 pad 1: /Project Architecture/LED/+LED_POWER -> +5V
- D61 pad 1: /Project Architecture/LED/+LED_POWER -> +5V
- D62 pad 1: /Project Architecture/LED/+LED_POWER -> +5V
- D63 pad 1: /Project Architecture/LED/+LED_POWER -> +5V
- D7 pad 1: /Project Architecture/LED/+LED_POWER -> +5V
- D8 pad 1: /Project Architecture/LED/+LED_POWER -> +5V
- D9 pad 1: /Project Architecture/LED/+LED_POWER -> +5V
- R21 pad 1: /Project Architecture/LED/+LED_POWER -> +5V
- R41 pad 1: /Project Architecture/LED/+LED_POWER -> +5V
- U10 pad 15: unconnected-(U10-IO3-Pad15) -> /Project Architecture/MCU/LED_DATA_LV
- U10 pad 33: Net-(U10-IO40) -> unconnected-(U10-IO40-Pad33)
- U12 pad 3: Net-(U10-IO40) -> /Project Architecture/MCU/LED_DATA_LV
- U4 pad 6: /Project Architecture/LED/+LED_POWER -> +5V
- U7 pad 6: /Project Architecture/LED/+LED_POWER -> +5V
- U9 pad 5: /Project Architecture/LED/+LED_POWER -> +5V
Routing:
- net +5V: track 0.00 -> 169.7 mm, vias 0 -> 60
- net /Project Architecture/LED/+LED_POWER: track 169.7 -> 0.00 mm
- net Net-(D37-DOUT): track 0.00 -> 74.9 mm, vias 0 -> 2
- net Net-(D29-DOUT): track 0.00 -> 74.9 mm, vias 0 -> 2
- net Net-(D46-DOUT): track 0.00 -> 67.0 mm, vias 0 -> 2
- net Net-(D20-DOUT): track 0.00 -> 66.6 mm, vias 0 -> 2
- net Net-(D53-DOUT): track 0.00 -> 59.1 mm, vias 0 -> 2
- net Net-(D13-DOUT): track 0.00 -> 58.2 mm, vias 0 -> 2
- net Net-(D60-DOUT): track 0.00 -> 42.4 mm, vias 0 -> 2
- net Net-(D6-DOUT): track 0.00 -> 41.6 mm, vias 0 -> 2
- net /Project Architecture/powerdelivery/+1.8V_CYPD: track 0.00 -> 14.7 mm
- net Net-(D33-DOUT): track 0.00 -> 12.5 mm
- net Net-(U9-FB): track 0.00 -> 9.47 mm
- net Net-(U3-VBUS_FET_EN): track 0.00 -> 8.93 mm
- net /Project Architecture/powerdelivery/USB_N: track 0.00 -> 8.10 mm, vias 0 -> 2
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- added copper zone on In1.Cu, net +5V
- added copper zone on B.Cu, net GND
- added copper zone on F.Cu, net GND
- added copper zone on In2.Cu, net GND
- added copper zone on F.Cu, net Net-(D2-K)
- added copper zone on F.Cu, net Net-(Q3-PadS)
Other:
- outline, holes or cut-outs redrawn
- board text removed: "PCB3D_BR_BOARDNAME"
- board text removed: "PCB3D_TL_BOARDNAME"

Commit message: PCB finished, export working
Parts:
- moved R40 14.7 mm to (104.3, 71.6), turned to -90 degrees
- moved R1 5.08 mm to (183.6, 44.4)
- moved R45 4.19 mm to (111.0, 79.9), turned to 0 degrees
- moved C35 2.48 mm to (106.8, 76.7)
- moved U8 2.47 mm to (106.8, 73.8)
- moved C2 2.32 mm to (187.8, 56.2), turned to 180 degrees
- moved C36 2.19 mm to (106.8, 70.8)
- moved R31 0.45 mm to (196.1, 74.8)
- moved R32 0.45 mm to (196.1, 77.8)
- moved R29 0.40 mm to (198.9, 101.7)
- moved C1 0.35 mm to (189.1, 46.9)
- moved R10 0.25 mm to (212.0, 94.2)
- moved R44 0.16 mm to (141.1, 25.9)
- turned R41 to 180 degrees
Connections:
- J2 pad SH: (no net) -> GND
- R45 pad 1: +3.3V -> VDDA
- R50 pad 1: VDDA -> +3.3V
- U13 pad 8: VDDA -> +3.3V
Routing:
- net /Project Architecture/LED/I2C_SCL: track 0.00 -> 169.4 mm, vias 0 -> 5
- net /Project Architecture/LED/I2C_SDA: track 0.00 -> 157.1 mm, vias 0 -> 4
- net +3.3V: track 0.00 -> 151.8 mm, vias 0 -> 4
- net /Project Architecture/powerdelivery/USB_P: track 6.90 -> 129.8 mm, vias 2 -> 4
- net /Project Architecture/powerdelivery/USB_N: track 8.10 -> 129.9 mm, vias 2 -> 4
- net /Project Architecture/MCU/Fault_PD: track 0.00 -> 95.5 mm, vias 0 -> 2
- net /Project Architecture/MCU/PG_PD: track 0.00 -> 92.9 mm, vias 0 -> 2
- net /Project Architecture/powerdelivery/+15V_VBUS: track 0.00 -> 83.5 mm, vias 0 -> 2
- net /Project Architecture/MCU/PD_INT: track 0.00 -> 77.2 mm, vias 0 -> 2
- net Net-(U10-IO12): track 0.00 -> 71.9 mm, vias 0 -> 4
- net /Project Architecture/MCU/PG_BAT: track 0.00 -> 69.6 mm, vias 0 -> 2
- net /Project Architecture/MCU/EN_DCDC_BAT: track 0.00 -> 62.0 mm, vias 0 -> 2
- net +5V: track 169.7 -> 224.9 mm, vias 60 -> 69
- net /Project Architecture/Power/+5V_SAFEPWR_IN: track 0.00 -> 53.7 mm
- net /Project Architecture/Battery/EN_CHG: track 0.00 -> 48.3 mm, vias 0 -> 4
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- added copper zone on F.Cu, net +3.3V
- added copper zone on B.Cu, net +5V
- added copper zone on F.Cu, net +5V
- added copper zone on In2.Cu, net +5V
- added copper zone on F.Cu, net /Project Architecture/Battery/+BAT_OUT
- added copper zone on F.Cu, net /Project Architecture/Power/+5V_BAT
- added copper zone on F.Cu, net /Project Architecture/Power/+5V_PD
- added copper zone on F.Cu, net /Project Architecture/powerdelivery/+15V_VBUS
- added copper zone on In1.Cu, net GND
- added copper zone on F.Cu, net Net-(C4-Pad1)
- added copper zone on F.Cu, net Net-(U3-VBUS_IN)
- added copper zone on In2.Cu, net Net-(U3-VBUS_IN)
- added copper zone on F.Cu, net Net-(U5-SW)
- added copper zone on F.Cu, net Net-(U6-SW)
- added copper zone on F.Cu, net Net-(U9-SW)
- removed copper zone on In1.Cu, net +5V
- removed copper zone on In2.Cu, net GND

Commit message: first Claude Software
Parts:
- added H1: MountingHole, MountingHole:MountingHole_2.7mm_M2.5, F.Cu at (101.0, 45.0)
- added H2: MountingHole, MountingHole:MountingHole_2.7mm_M2.5, F.Cu at (201.1, 45.0)
- added H3: MountingHole, MountingHole:MountingHole_2.7mm_M2.5, F.Cu at (201.1, 125.0)
- added H4: MountingHole, MountingHole:MountingHole_2.7mm_M2.5, F.Cu at (101.0, 125.0)
- C37: value 100n -> 100nF
- L1: value 2.2u -> 2.2uH
Routing:
- net /Project Architecture/powerdelivery/USB_P: track 129.8 -> 132.2 mm, vias 4 -> 3
- net /Project Architecture/powerdelivery/USB_N: track 129.9 -> 131.4 mm, vias 4 -> 3
- net GND: vias 207 -> 353
