File: Hardware/Electrical/PCB_v2/Power.kicad_sch (KiCad schematic)
At the start: 65 parts, among them U4 LM73100RPWR, U5 TPS51385, U6 TPS61022, U7 LM73100RPWR, U8 TLV77333PDBVR, U9 LMR50410

Commit message: Components placed
Parts:
- C15, C18, C23, C29, C34, C40, C43: value 100n -> 100nF
- C16, C19, C20, C21, C27, C30, C31, C32: value 22u -> 22uF
- C17, C22, C26, C28, C33, C35, C36: value 1u -> 1uF
- C38, C39, C42: value 2.2u -> 2.2uF
- C41: value 10u -> 10uF
- D3: footprint (none) -> Package_TO_SOT_SMD:SOT-23; *LCSC Part Number (none) -> C2135; LCSC Part # (none) -> C2135
- R29: value 0 -> 0 Ohm
- U8: *LCSC Part Number (none) -> C32445874
Connections:
- net +5V: now also C38.1, C39.1, C40.1, D3.3 (K), R21.1, R41.1, U4.6 (OUT), U7.6 (OUT), U9.5 (VIN)
- net +5V_SAFEPWR_IN: now also D3.1 (A)
- removed net +5V_Uninterrupted_out: C38.1, C39.1, C40.1, D3.1 (K), R21.1, R41.1, U4.6 (OUT), U7.6 (OUT), U9.5 (VIN)

Commit message: first Claude Software
Parts:
- C15, C18, C23, C29, C34, C40, C43: LCSC Part # (none) -> C14663
- C16, C19, C20, C21, C27, C30, C31, C32: LCSC Part # (none) -> C12891
- C17, C22, C26, C28, C33, C35, C36: *LCSC Part Number C1848 -> C15849; LCSC Part # (none) -> C15849
- C24: LCSC Part # (none) -> C1653
- C37: value 100n -> 100nF; LCSC Part # (none) -> C14663
- C38, C39, C42: LCSC Part # (none) -> C23630
- C41: LCSC Part # (none) -> C13585
- L2, L3: LCSC Part # (none) -> C2847480
- L4: LCSC Part # (none) -> C553980
- R18: LCSC Part # (none) -> C23196
- R19: LCSC Part # (none) -> C23197
- R20, R34: LCSC Part # (none) -> C137765
- R21, R31: LCSC Part # (none) -> C137684
- R22: LCSC Part # (none) -> C22807
- R23, R36: LCSC Part # (none) -> C137694
- R24, R37: LCSC Part # (none) -> C23024
- R25, R30, R32, R39: *LCSC Part Number C137684 -> C23265; LCSC Part # (none) -> C23265
- R26, R28, R35, R38: LCSC Part # (none) -> C25803
- R27: LCSC Part # (none) -> C4184
- R33: LCSC Part # (none) -> C246003
- R40, R41: LCSC Part # (none) -> C25804
- R42: LCSC Part # (none) -> C22783
- R43: LCSC Part # (none) -> C23184
- U4, U7: LCSC Part # (none) -> C3210761
- U5: LCSC Part # (none) -> C22418767
- U6: *LCSC Part Number TPS61022RWUR -> C915088; LCSC Part # (none) -> C915088
- U8: LCSC Part # (none) -> C32445874
- U9: LCSC Part # (none) -> C2841056
