File: Hardware/Electrical/PCB_v2/Project Architecture.kicad_sch (KiCad schematic)
At the start: 0 parts

Commit message: manual LED circle done
Other:
- sheet Section A - Title A renamed Battery
- added sheet LED (LED.kicad_sch)
- added sheet MCU (MCU.kicad_sch)
- added sheet Power (Power.kicad_sch)
- added sheet powerdelivery (powerdelivery.kicad_sch)
- sheet Battery: file Section A - Title A.kicad_sch -> Battery.kicad_sch
- sheet Battery ports: added +BAT_OUT, +CHG_IN, EN_CHG; removed none
- note removed: "Page 4"

Commit message: first Claude Software
Parts:
- added H1, H2, H3, H4: MountingHole, MountingHole:MountingHole_2.7mm_M2.5, symbol Mechanical:MountingHole
