File: Hardware/Electrical/PCB_v2/PCB_v2.kicad_sch (KiCad schematic)
At the start: 0 parts

Commit message: first fully working software, undervoltage not added yet
Other:
- note removed: "${VARIANT} ${RELEASE_DATE}"
- note removed: "Add a comment here"
- note removed: "CHECKED - There shouldn't be any mistakes. Contact the engineer if you find any."
- note removed: "DESIGN CONSIDERATIONS"
- note removed: "DRAFT - Very early stage of schematic, ignore details."
- note removed: "NOTES"
- note removed: "Not fitted components are marked as"
- note removed: "PRELIMINARY - Close to final schematic."
- note removed: "RELEASED - A board with this schematic has been sent to production."
